File: hardware/hardware.kicad_pcb (KiCad board)
At the start: 2 copper layers, 108 x 54 mm, 3 parts, among them J2 Pinouts, J4 AVR-ISP-6, U1 ATmega8A-A

Commit message: organized
Parts:
- added Y1: 16Mhz, Crystal:Resonator_SMD_Murata_CSTxExxV-3Pin_3.0x1.1mm_HandSoldering, F.Cu at (168.1, 79.5)
Connections:
- U1 pad 7: unconnected-(U1-PB6/XTAL1-Pad7) -> Net-(U1-PB6/XTAL1)
- U1 pad 8: unconnected-(U1-PB7/XTAL2-Pad8) -> Net-(U1-PB7/XTAL2)
Routing:
- net Net-(U1-PB7/XTAL2): track 0.00 -> 5.58 mm
- net GND: track 155.1 -> 160.7 mm
- net Net-(U1-PB6/XTAL1): track 0.00 -> 3.86 mm
