File: hardware/hardware.kicad_sch (KiCad schematic)
At the start: 4 parts, among them J1 Connector, J2 Pinouts, J4 AVR-ISP-6, U1 ATmega8A-A

Commit message: organized
Parts:
- added Y1: 16Mhz, Crystal:Resonator_SMD_Murata_CSTxExxV-3Pin_3.0x1.1mm_HandSoldering, symbol Device:Resonator
Connections:
- net GND: now also Y1.2
- net at U1.7 (PB6/XTAL1): now also Y1.1
- net at U1.8 (PB7/XTAL2): now also Y1.3
- no-connect marks 16 -> 14
Changed lines of the file:
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@@
-	)
-	(no_connect
-		(at 132.08 64.77)
 	)
 	(no_connect
@@
 	)
 	(no_connect
-		(at 132.08 59.69)
-	)
-	(no_connect
 		(at 162.56 90.17)
 	)
@@
 	(no_connect
 		(at 162.56 59.69)
+	)
+	(wire
+		(pts
+			(xy 129.54 57.15) (xy 115.57 57.15)
+		)
+		(stroke
+			(width 0)
+			(type default)
+		)
 	)
 	(wire
@@
 	(wire
 		(pts
-			(xy 147.32 118.11) (xy 149.86 118.11)
+			(xy 129.54 59.69) (xy 129.54 57.15)
 		)
 		(stroke
@@
 	(wire
 		(pts
-			(xy 147.32 46.99) (xy 149.86 46.99)
+			(xy 147.32 118.11) (xy 149.86 118.11)
 		)
 		(stroke
@@
 	(wire
 		(pts
+			(xy 147.32 46.99) (xy 149.86 46.99)
+		)
+		(stroke
+			(width 0)
+			(type default)
+		)
+	)
+	(wire
+		(pts
 			(xy 147.32 45.72) (xy 147.32 46.99)
+		)
+		(stroke
+			(width 0)
+			(type default)
+		)
+	)
+	(wire
+		(pts
+			(xy 115.57 64.77) (xy 132.08 64.77)
+		)
+		(stroke
+			(width 0)
+			(type default)
+		)
+	)
+	(wire
+		(pts
+			(xy 109.22 60.96) (xy 110.49 60.96)
+		)
+		(stroke
+			(width 0)
+			(type default)
+		)
+	)
+	(wire
+		(pts
+			(xy 132.08 59.69) (xy 129.54 59.69)
 		)
 		(stroke
@@
 		)
 		(instances
-			(project "SLE4442-Emulator"
+			(project "hardware"
 				(path "/79b7f5d6-5330-4d70-822f-eb7b03666395"
 					(reference "U1")
@@
 		)
 		(instances
-			(project "SLE4442-Emulator"
+			(project "hardware"
 				(path "/79b7f5d6-5330-4d70-822f-eb7b03666395"
 					(reference "#PWR04")
@@
 		)
 		(instances
-			(project "SLE4442-Emulator"
+			(project "hardware"
 				(path "/79b7f5d6-5330-4d70-822f-eb7b03666395"
 					(reference "#FLG01")
@@
 		)
 		(instances
-			(project "SLE4442-Emulator"
+			(project "hardware"
 				(path "/79b7f5d6-5330-4d70-822f-eb7b03666395"
 					(reference "J1")
@@
 		)
 		(instances
-			(project "SLE4442-Emulator"
+			(project "hardware"
 				(path "/79b7f5d6-5330-4d70-822f-eb7b03666395"
 					(reference "J2")
@@
 		)
 		(instances
-			(project "SLE4442-Emulator"
+			(project "hardware"
 				(path "/79b7f5d6-5330-4d70-822f-eb7b03666395"
 					(reference "#FLG02")
@@
 		)
 		(instances
-			(project "SLE4442-Emulator"
+			(project "hardware"
 				(path "/79b7f5d6-5330-4d70-822f-eb7b03666395"
 					(reference "#PWR02")
@@
 		)
 		(instances
-			(project "SLE4442-Emulator"
+			(project "hardware"
 				(path "/79b7f5d6-5330-4d70-822f-eb7b03666395"
 					(reference "J4")
+					(unit 1)
+				)
+			)
+		)
+	)
+	(symbol
+		(lib_id "power:GND")
+		(at 109.22 60.96 0)
+		(unit 1)
+		(body_style 1)
+		(exclude_from_sim no)
+		(in_bom yes)
+		(on_board yes)
+		(in_pos_files yes)
+		(dnp no)
+		(fields_autoplaced yes)
+		(property "Reference" "#PWR010"
+			(at 109.22 67.31 0)
+			(hide yes)
+			(show_name no)
+			(do_not_autoplace no)
+			(effects
+				(font
+					(size 1.27 1.27)
+				)
+			)
+		)
+		(property "Value" "GND"
+			(at 109.22 66.04 0)
+			(show_name no)
+			(do_not_autoplace no)
+			(effects
+				(font
+					(size 1.27 1.27)
+				)
+			)
+		)
+		(property "Footprint" ""
+			(at 109.22 60.96 0)
+			(hide yes)
+			(show_name no)
+			(do_not_autoplace no)
+			(effects
+				(font
+					(size 1.27 1.27)
+				)
+			)
+		)
+		(property "Datasheet" ""
+			(at 109.22 60.96 0)
+			(hide yes)
+			(show_name no)
+			(do_not_autoplace no)
+			(effects
+				(font
+					(size 1.27 1.27)
+				)
+			)
+		)
+		(property "Description" "Power symbol creates a global label with name \"GND\" , ground"
+			(at 109.22 60.96 0)
+			(hide yes)
+			(show_name no)
+			(do_not_autoplace no)
+			(effects
+				(font
+					(size 1.27 1.27)
+				)
+			)
+		)
+		(pin "1"
+		)
+		(instances
+			(project "hardware"
+				(path "/79b7f5d6-5330-4d70-822f-eb7b03666395"
+					(reference "#PWR010")
 					(unit 1)
 				)
@@
 		)
 		(instances
-			(project "SLE4442-Emulator"
+			(project "hardware"
 				(path "/79b7f5d6-5330-4d70-822f-eb7b03666395"
 					(reference "#PWR03")
@@
 		)
 		(instances
-			(project "SLE4442-Emulator"
+			(project "hardware"
 				(path "/79b7f5d6-5330-4d70-822f-eb7b03666395"
 					(reference "#PWR08")
@@
 		)
 		(instances
-			(project "SLE4442-Emulator"
+			(project "hardware"
 				(path "/79b7f5d6-5330-4d70-822f-eb7b03666395"
 					(reference "#PWR05")
+					(unit 1)
+				)
+			)
+		)
+	)
+	(symbol
+		(lib_id "Device:Resonator")
+		(at 115.57 60.96 270)
+		(unit 1)
+		(body_style 1)
+		(exclude_from_sim no)
+		(in_bom yes)
+		(on_board yes)
+		(in_pos_files yes)
+		(dnp no)
+		(fields_autoplaced yes)
+		(property "Reference" "Y1"
+			(at 119.38 59.6899 90)
+			(show_name no)
+			(do_not_autoplace no)
+			(effects
+				(font
+					(size 1.27 1.27)
+				)
+				(justify left)
+			)
+		)
+		(property "Value" "16Mhz"
+			(at 119.38 62.2299 90)
+			(show_name no)
+			(do_not_autoplace no)
+			(effects
+				(font
+					(size 1.27 1.27)
+				)
+				(justify left)
+			)
+		)
+		(property "Footprint" "Crystal:Resonator_SMD_Murata_CSTxExxV-3Pin_3.0x1.1mm_HandSoldering"
+			(at 115.57 60.325 0)
+			(hide yes)
+			(show_name no)
+			(do_not_autoplace no)
+			(effects
+				(font
+					(size 1.27 1.27)
+				)
+			)
+		)
+		(property "Datasheet" ""
+			(at 115.57 60.325 0)
+			(hide yes)
+			(show_name no)
+			(do_not_autoplace no)
+			(effects
+				(font
+					(size 1.27 1.27)
+				)
+			)
+		)
+		(property "Description" "Three pin ceramic resonator"
+			(at 115.57 60.96 0)
+			(hide yes)
+			(show_name no)
+			(do_not_autoplace no)
+			(effects
+				(font
+					(size 1.27 1.27)
+				)
+			)
+		)
+		(pin "1"
+		)
+		(pin "3"
+		)
+		(pin "2"
+		)
+		(instances
+			(project "hardware"
+				(path "/79b7f5d6-5330-4d70-822f-eb7b03666395"
+					(reference "Y1")
 					(unit 1)
 				)
@@
 		)
 		(instances
-			(project "SLE4442-Emulator"
+			(project "hardware"
 				(path "/79b7f5d6-5330-4d70-822f-eb7b03666395"
 					(reference "#PWR06")
@@
 		)
 		(instances
-			(project "SLE4442-Emulator"
+			(project "hardware"
 				(path "/79b7f5d6-5330-4d70-822f-eb7b03666395"
 					(reference "#PWR09")
@@
 		)
 		(instances
-			(project "SLE4442-Emulator"
+			(project "hardware"
 				(path "/79b7f5d6-5330-4d70-822f-eb7b03666395"
 					(reference "#PWR01")
@@
 		)
 		(instances
-			(project "SLE4442-Emulator"
+			(project "hardware"
 				(path "/79b7f5d6-5330-4d70-822f-eb7b03666395"
 					(reference "#PWR07")

Commit message: update bom
Parts:
- U1: LCSC Part # (none) -> C16190; MPN (none) -> ATMEGA8A-AU
- Y1: LCSC Part # (none) -> C32180; MPN (none) -> CSTCE16M0V53-R0
Changed lines of the file:
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@@
+			)
+		)
+		(property "LCSC Part #" "C16190"
+			(at 147.32 82.55 0)
+			(hide yes)
+			(show_name no)
+			(do_not_autoplace no)
+			(effects
+				(font
+					(size 1.27 1.27)
+				)
+			)
+		)
+		(property "MPN" "ATMEGA8A-AU"
+			(at 147.32 82.55 0)
+			(hide yes)
+			(show_name no)
+			(do_not_autoplace no)
+			(effects
+				(font
+					(size 1.27 1.27)
+				)
 			)
 		)
@@
 			(at 115.57 60.96 0)
 			(hide yes)
+			(show_name no)
+			(do_not_autoplace no)
+			(effects
+				(font
+					(size 1.27 1.27)
+				)
+			)
+		)
+		(property "LCSC Part #" "C32180"
+			(at 115.57 60.96 0)
+			(hide yes)
+			(show_name no)
+			(do_not_autoplace no)
+			(effects
+				(font
+					(size 1.27 1.27)
+				)
+			)
+		)
+		(property "MPN" "CSTCE16M0V53-R0"
+			(at 115.57 60.96 0)
+			(hide yes)
